File: Conejo.kicad_sch (KiCad schematic)
At the start: 2 parts

Commit message: feat(pcb): Version 1.0.0
- Change decoupling capacitors from 4.7uF/1uF pairs to both 4.7uF
Parts:
- G1, G2: value (none) -> LOGO; footprint (none) -> Conejo:Powered_By_ZMK (Large)
Changed lines of the file:
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@@
       (effects (font (size 1.27 1.27)) hide)
     )
-    (property "Value" "" (id 1) (at 114.3 69.0412 0)
-      (effects (font (size 1.27 1.27)) hide)
-    )
-    (property "Footprint" "" (id 2) (at 114.3 66.675 0)
+    (property "Value" "LOGO" (id 1) (at 114.3 69.0412 0)
+      (effects (font (size 1.27 1.27)) hide)
+    )
+    (property "Footprint" "Conejo:Powered_By_ZMK (Large)" (id 2) (at 114.3 66.675 0)
       (effects (font (size 1.27 1.27)) hide)
     )
@@
       (effects (font (size 1.27 1.27)) hide)
     )
-    (property "Value" "" (id 1) (at 114.3 69.0412 0)
-      (effects (font (size 1.27 1.27)) hide)
-    )
-    (property "Footprint" "" (id 2) (at 114.3 66.675 0)
+    (property "Value" "LOGO" (id 1) (at 114.3 69.0412 0)
+      (effects (font (size 1.27 1.27)) hide)
+    )
+    (property "Footprint" "Conejo:Powered_By_ZMK (Large)" (id 2) (at 114.3 66.675 0)
       (effects (font (size 1.27 1.27)) hide)
     )
@@
     )
     (path "/1803c616-4a91-454a-85d9-d17a70de9e60/e83e3453-2fd4-4b68-868a-d2a11761891e"
-      (reference "C2") (unit 1) (value "1uF") (footprint "Capacitor_SMD:C_0402_1005Metric")
+      (reference "C2") (unit 1) (value "4u7F") (footprint "Capacitor_SMD:C_0402_1005Metric")
     )
     (path "/1803c616-4a91-454a-85d9-d17a70de9e60/5ee4cdbb-1860-47a0-8dda-97cdb367591d"
-      (reference "C3") (unit 1) (value "1uF") (footprint "Capacitor_SMD:C_0402_1005Metric")
+      (reference "C3") (unit 1) (value "4u7F") (footprint "Capacitor_SMD:C_0402_1005Metric")
     )
     (path "/1803c616-4a91-454a-85d9-d17a70de9e60/9c911103-9838-4680-a02e-10f670092c7c"
@@
     )
     (path "/1803c616-4a91-454a-85d9-d17a70de9e60/b48cec1d-e281-4381-8fa7-0bbcb8b720ea"
-      (reference "C7") (unit 1) (value "1uF") (footprint "Capacitor_SMD:C_0402_1005Metric")
+      (reference "C7") (unit 1) (value "4u7F") (footprint "Capacitor_SMD:C_0402_1005Metric")
     )
     (path "/a6c855a7-3fa9-426b-8144-57b4803ad800/39ca6f2c-d0f7-47e3-be39-6dd3edca81b9"
