File: USB-C.kicad_sch (KiCad schematic)
At the start: 6 parts, among them J2 HRO_TYPE-C-31-M-12, U3 SRV05-4

Commit message: feat(pcb): Version 0.4.1
- Add oscilloscope probing pads/labels
Connections:
- no-connect marks 2 -> 4
Changed lines of the file:
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@@
   )
   (no_connect (at 41.91 60.325))
+  (no_connect (at 117.475 43.18))
+  (no_connect (at 92.075 48.26))
   (no_connect (at 41.91 57.785))
   (polyline (pts (xy 127 25.4) (xy 127 66.675))

Commit message: feat(pcb): Switch from 4.3mm NPTH mounting holes to M2 PTH
Parts:
- F2: value 500mA -> (none); footprint Fuse:Fuse_0603_1608Metric -> (none)
- FB1: value 120R@100MHz -> (none); footprint Inductor_SMD:L_0402_1005Metric -> (none)
- J2: value HRO_TYPE-C-31-M-12 -> (none); footprint Conejo:USB_C_Receptacle_HRO_TYPE-C-31-M-12 (Reversible) -> (none)
- R8, R9: value 5K1 -> (none); footprint Resistor_SMD:R_0402_1005Metric -> (none)
- U3: value SRV05-4 -> (none); footprint marbastlib-various:SOT-23-6-routable -> (none)
Changed lines of the file:
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@@
       (effects (font (size 1.27 1.27)) (justify left))
     )
-    (property "Value" "SRV05-4" (id 1) (at 107.5437 34.3971 0)
+    (property "Value" "" (id 1) (at 107.5437 34.3971 0)
       (effects (font (size 1.27 1.27)) (justify left))
     )
-    (property "Footprint" "marbastlib-various:SOT-23-6-routable" (id 2) (at 122.555 57.15 0)
+    (property "Footprint" "" (id 2) (at 122.555 57.15 0)
       (effects (font (size 1.27 1.27)) hide)
     )
@@
       (effects (font (size 1.27 1.27)) (justify left))
     )
-    (property "Value" "5K1" (id 1) (at 71.3486 42.9772 0)
+    (property "Value" "" (id 1) (at 71.3486 42.9772 0)
       (effects (font (size 1.27 1.27)) (justify left))
     )
-    (property "Footprint" "Resistor_SMD:R_0402_1005Metric" (id 2) (at 69.85 41.275 0)
+    (property "Footprint" "" (id 2) (at 69.85 41.275 0)
       (effects (font (size 1.27 1.27)) hide)
     )
@@
       (effects (font (size 1.27 1.27)) (justify right))
     )
-    (property "Value" "5K1" (id 1) (at 62.0014 42.9772 0)
+    (property "Value" "" (id 1) (at 62.0014 42.9772 0)
       (effects (font (size 1.27 1.27)) (justify right))
     )
-    (property "Footprint" "Resistor_SMD:R_0402_1005Metric" (id 2) (at 63.5 41.275 0)
+    (property "Footprint" "" (id 2) (at 63.5 41.275 0)
       (effects (font (size 1.27 1.27)) hide)
     )
@@
     (in_bom yes) (on_board yes) (fields_autoplaced)
     (property "Reference" "F2" (id 0) (at 50.8 25.2562 90))
-    (property "Value" "500mA" (id 1) (at 50.8 27.7931 90))
-    (property "Footprint" "Fuse:Fuse_0603_1608Metric" (id 2) (at 55.88 28.575 0)
+    (property "Value" "" (id 1) (at 50.8 27.7931 90))
+    (property "Footprint" "" (id 2) (at 55.88 28.575 0)
       (effects (font (size 1.27 1.27)) (justify left) hide)
     )
@@
     (in_bom yes) (on_board yes) (fields_autoplaced)
     (property "Reference" "J2" (id 0) (at 26.67 23.6052 0))
-    (property "Value" "HRO_TYPE-C-31-M-12" (id 1) (at 26.67 26.1421 0))
-    (property "Footprint" "Conejo:USB_C_Receptacle_HRO_TYPE-C-31-M-12 (Reversible)" (id 2) (at 30.48 45.085 0)
+    (property "Value" "" (id 1) (at 26.67 26.1421 0))
+    (property "Footprint" "" (id 2) (at 30.48 45.085 0)
       (effects (font (size 1.27 1.27)) hide)
     )
@@
     (in_bom yes) (on_board yes) (fields_autoplaced)
     (property "Reference" "FB1" (id 0) (at 63.4619 24.4434 90))
-    (property "Value" "120R@100MHz" (id 1) (at 63.4619 26.9803 90))
-    (property "Footprint" "Inductor_SMD:L_0402_1005Metric" (id 2) (at 63.5 31.623 90)
+    (property "Value" "" (id 1) (at 63.4619 26.9803 90))
+    (property "Footprint" "" (id 2) (at 63.5 31.623 90)
       (effects (font (size 1.27 1.27)) hide)
     )

Commit message: feat(pcb): Version 1.0.0
- Change decoupling capacitors from 4.7uF/1uF pairs to both 4.7uF
Parts:
- F2: value (none) -> 500mA; footprint (none) -> Fuse:Fuse_0603_1608Metric
- FB1: value (none) -> 120R@100MHz; footprint (none) -> Inductor_SMD:L_0402_1005Metric
- J2: value (none) -> HRO_TYPE-C-31-M-12; footprint (none) -> Conejo:USB_C_Receptacle_HRO_TYPE-C-31-M-12 (Reversible)
- R8, R9: value (none) -> 5K1; footprint (none) -> Resistor_SMD:R_0402_1005Metric
- U3: value (none) -> SRV05-4; footprint (none) -> marbastlib-various:SOT-23-6-routable
Changed lines of the file:
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@@
       (effects (font (size 1.27 1.27)) (justify left))
     )
-    (property "Value" "" (id 1) (at 107.5437 34.3971 0)
+    (property "Value" "SRV05-4" (id 1) (at 107.5437 34.3971 0)
       (effects (font (size 1.27 1.27)) (justify left))
     )
-    (property "Footprint" "" (id 2) (at 122.555 57.15 0)
+    (property "Footprint" "marbastlib-various:SOT-23-6-routable" (id 2) (at 122.555 57.15 0)
       (effects (font (size 1.27 1.27)) hide)
     )
@@
       (effects (font (size 1.27 1.27)) (justify left))
     )
-    (property "Value" "" (id 1) (at 71.3486 42.9772 0)
+    (property "Value" "5K1" (id 1) (at 71.3486 42.9772 0)
       (effects (font (size 1.27 1.27)) (justify left))
     )
-    (property "Footprint" "" (id 2) (at 69.85 41.275 0)
+    (property "Footprint" "Resistor_SMD:R_0402_1005Metric" (id 2) (at 69.85 41.275 0)
       (effects (font (size 1.27 1.27)) hide)
     )
@@
       (effects (font (size 1.27 1.27)) (justify right))
     )
-    (property "Value" "" (id 1) (at 62.0014 42.9772 0)
+    (property "Value" "5K1" (id 1) (at 62.0014 42.9772 0)
       (effects (font (size 1.27 1.27)) (justify right))
     )
-    (property "Footprint" "" (id 2) (at 63.5 41.275 0)
+    (property "Footprint" "Resistor_SMD:R_0402_1005Metric" (id 2) (at 63.5 41.275 0)
       (effects (font (size 1.27 1.27)) hide)
     )
@@
     (in_bom yes) (on_board yes) (fields_autoplaced)
     (property "Reference" "F2" (id 0) (at 50.8 25.2562 90))
-    (property "Value" "" (id 1) (at 50.8 27.7931 90))
-    (property "Footprint" "" (id 2) (at 55.88 28.575 0)
+    (property "Value" "500mA" (id 1) (at 50.8 27.7931 90))
+    (property "Footprint" "Fuse:Fuse_0603_1608Metric" (id 2) (at 55.88 28.575 0)
       (effects (font (size 1.27 1.27)) (justify left) hide)
     )
@@
     (in_bom yes) (on_board yes) (fields_autoplaced)
     (property "Reference" "J2" (id 0) (at 26.67 23.6052 0))
-    (property "Value" "" (id 1) (at 26.67 26.1421 0))
-    (property "Footprint" "" (id 2) (at 30.48 45.085 0)
+    (property "Value" "HRO_TYPE-C-31-M-12" (id 1) (at 26.67 26.1421 0))
+    (property "Footprint" "Conejo:USB_C_Receptacle_HRO_TYPE-C-31-M-12 (Reversible)" (id 2) (at 30.48 45.085 0)
       (effects (font (size 1.27 1.27)) hide)
     )
@@
     (in_bom yes) (on_board yes) (fields_autoplaced)
     (property "Reference" "FB1" (id 0) (at 63.4619 24.4434 90))
-    (property "Value" "" (id 1) (at 63.4619 26.9803 90))
-    (property "Footprint" "" (id 2) (at 63.5 31.623 90)
+    (property "Value" "120R@100MHz" (id 1) (at 63.4619 26.9803 90))
+    (property "Footprint" "Inductor_SMD:L_0402_1005Metric" (id 2) (at 63.5 31.623 90)
       (effects (font (size 1.27 1.27)) hide)
     )
